File: audio.kicad_sch (KiCad schematic)
At the start: 6 parts, among them J1 USB4105-GF-A, U1 PCM5102APW, U2 TPA6130A2RTJR, U3 DEV-15583

Commit message: vähän lisää piirtelin
Parts:
- added C10, C5, C6: C_Polarized_US, symbol Device:C_Polarized_US
- added C3, C4, C7, C9: C, symbol Device:C
- added C8: 2.2u, symbol Device:C
Connections:
- net GND: now also U1.16 (FMT), U1.18 (LDOO), C4.2, C5.1
- net 3.3VA: now reaches U1.1 (CPVDD)
- net 3.3VA: now also C10.1, C9.2
- net PCM Audio Source: now reaches U1.12 (SCK)
- net PCM Audio Source: now also U1.13 (BCK), U1.14 (DIN), U1.15 (LRCK)
- net mute circuit: now reaches U1.17 (XSMT)
- net at U1.19 (DGND): now also C3.1, C4.1, C5.2, C6.1
- net at U1.2 (CAPP): now also C8.1
- net 3.3V: now reaches U1.20 (DVDD)
- net 3.3V: now also C3.2, C6.2
- net at U1.3 (CPGND): now also C10.2, C7.2, C9.1
- net at U1.4 (CAPM): now also C8.2
- net at U1.5 (VNEG): now also C7.1

Commit message: PCM circuit done
Parts:
- added C11, C12: C, symbol Device:C
- added R1, R2: R, symbol Device:R
Connections:
- net at U1.6 (OUTL): now also R1.1
- net at U1.7 (OUTR): now also R2.1
- new net AGND: C11.1, C12.2
- new net Left Channel Line Output: C11.2, R1.2
- new net Right Channel Line Output: C12.1, R2.2

Commit message: Amplifier reference values
Parts:
- added C13, C14: C, symbol Device:C
- added R3, R4: R, symbol Device:R
Connections:
- net AGND: now also R3.1, R4.1
- net Left Channel Line Output: now also U2.1 (LEFTINM)
- net Right Channel Line Output: now also U2.5 (RIGHTINM)
- net at U2.2 (LEFTINP): now also C14.2
- net at U2.4 (RIGHTINP): now also C13.2
- new net: C14.1, R4.2
- new net: C13.1, R3.2

Commit message: Amplifier stuff
Parts:
- added C15, C16, C17, C18: C_Polarized_US, symbol Device:C_Polarized_US
Connections:
- net GND: now also U2.13 (GND), U2.19 (GND), C16.1, C17.2, C18.2
- net at U2.12 (VDD): now also C18.1
- net at U2.16 (CPVSS): now also C16.2
- net at U2.17 (CPN): now also C15.2
- net at U2.18 (CPP): now also C15.1
- net at U2.20 (VDD): now also C17.1
